File: GameBoardMatrix/hardware/GameBoardMatrix/GameBoardMatrix.kicad_sch (KiCad schematic)
At the start: 1 part

Commit message: Started on PCB/Schematic Design
Parts:
- removed C1: C, ECE445L:C_Axial_200mil, symbol ECE445L:C
- added J1: RPI_5_HeaderPins, Connector_PinSocket_2.54mm:PinSocket_2x20_P2.54mm_Vertical, symbol Connector_Generic:Conn_02x20_Odd_Even
- added U1, U2, U3, U4, U5: MUX, D16, symbol 8to1_MUX:SN74HC151DR
- added U6, U7, U8: A3144, A3144HallEffect:1x03_P1.50mm_Vertical_A3144HallEffect, symbol Sensor_Magnetic:A1104LLHL
Other:
- note added: "Hall Effect Matrix Game Board-Senior Design"

Commit message: Finished most of the schematic
Still need to tie outputs to gpio pins
Parts:
- added U10, U11, U12, U13, U14, U15, U16, U17, U18, U19, U20, U21, U22, U23, U24, U25, U26, U27, U28, U29, U30, U31, U32, U33, U34, U35, U36, U37, U38, U39, U40, U41, U42, U43, U44, U45, U9: A3144, A3144HallEffect:1x03_P1.50mm_Vertical_A3144HallEffect, symbol Sensor_Magnetic:A1104LLHL
Connections:
- net at U4.1 (D3): now also U39.2 (VOUT)
- net GPIO15/PIN10: now reaches U4.10 (B)
- net GPIO15/PIN10: now also J1.10 (GPIO15), U1.10 (B), U2.10 (B), U3.10 (B), U5.10 (B)
- net GPIO14/PIN8: now reaches U4.11 (A)
- net GPIO14/PIN8: now also J1.8 (GPIO14), U1.11 (A), U2.11 (A), U3.11 (A), U5.11 (A)
- net at U4.12 (D7): now also U40.2 (VOUT)
- net at U4.13 (D6): now also U31.2 (VOUT)
- net at U4.14 (D5): now also U22.2 (VOUT)
- net at U4.15 (D4): now also U13.2 (VOUT)
- net 3.3V_Board: now reaches U4.16 (VCC)
- net 3.3V_Board: now also J1.1 (3.3V), U1.16 (VCC), U2.16 (VCC), U3.16 (VCC), U5.16 (VCC), U6.1 (VCC), U7.1 (VCC), U8.1 (VCC), U10.1 (VCC), U11.1 (VCC), U12.1 (VCC), U13.1 (VCC), U14.1 (VCC), U15.1 (VCC), U16.1 (VCC), U17.1 (VCC), U18.1 (VCC), U19.1 (VCC), U20.1 (VCC), U21.1 (VCC), U22.1 (VCC), U23.1 (VCC), U24.1 (VCC), U25.1 (VCC), U26.1 (VCC), U27.1 (VCC), U28.1 (VCC), U29.1 (VCC), U30.1 (VCC), U31.1 (VCC), U32.1 (VCC), U33.1 (VCC), U34.1 (VCC), U35.1 (VCC), U36.1 (VCC), U37.1 (VCC), U38.1 (VCC), U39.1 (VCC), U40.1 (VCC), U41.1 (VCC), U42.1 (VCC), U43.1 (VCC), U44.1 (VCC), U45.1 (VCC), U9.1 (VCC)
- net at U4.2 (D2): now also U30.2 (VOUT)
- net at U4.3 (D1): now also U21.2 (VOUT)
- net at U4.4 (D0): now also U12.2 (VOUT)
- net GND: now reaches U4.7 (*G)
- net GND: now also U1.7 (*G), U1.8 (GND), U2.7 (*G), U2.8 (GND), U3.7 (*G), U3.8 (GND), U4.8 (GND), U5.8 (GND), U6.3 (GND), U7.3 (GND), U8.3 (GND), U10.3 (GND), U11.3 (GND), U12.3 (GND), U13.3 (GND), U14.3 (GND), U15.3 (GND), U16.3 (GND), U17.3 (GND), U18.3 (GND), U19.3 (GND), U20.3 (GND), U21.3 (GND), U22.3 (GND), U23.3 (GND), U24.3 (GND), U25.3 (GND), U26.3 (GND), U27.3 (GND), U28.3 (GND), U29.3 (GND), U30.3 (GND), U31.3 (GND), U32.3 (GND), U33.3 (GND), U34.3 (GND), U35.3 (GND), U36.3 (GND), U37.3 (GND), U38.3 (GND), U39.3 (GND), U40.3 (GND), U41.3 (GND), U42.3 (GND), U43.3 (GND), U44.3 (GND), U45.3 (GND), U9.3 (GND)
- net GPIO18/PIN12: now reaches U4.9 (C)
- net GPIO18/PIN12: now also J1.12 (GPIO18), U1.9 (C), U2.9 (C), U3.9 (C), U5.9 (C)
- net at U2.1 (D3): now also U35.2 (VOUT)
- net at U2.12 (D7): now also U36.2 (VOUT)
- net at U2.13 (D6): now also U27.2 (VOUT)
- net at U2.14 (D5): now also U18.2 (VOUT)
- net at U2.15 (D4): now also U9.2 (VOUT)
- net at U2.2 (D2): now also U26.2 (VOUT)
- net at U2.3 (D1): now also U17.2 (VOUT)
- net at U2.4 (D0): now also U8.2 (VOUT)
- net at U7.2 (VOUT): now also U1.15 (D4)
- net at U6.2 (VOUT): now also U1.4 (D0)
- net at U3.1 (D3): now also U37.2 (VOUT)
- net at U3.12 (D7): now also U38.2 (VOUT)
- net at U3.13 (D6): now also U29.2 (VOUT)
- net at U3.14 (D5): now also U20.2 (VOUT)
- net at U3.15 (D4): now also U11.2 (VOUT)
- net at U3.2 (D2): now also U28.2 (VOUT)
- net at U3.3 (D1): now also U19.2 (VOUT)
- net at U3.4 (D0): now also U10.2 (VOUT)
- net at U5.1 (D3): now also U41.2 (VOUT)
- net at U5.12 (D7): now also U45.2 (VOUT)
- net at U5.13 (D6): now also U44.2 (VOUT)
- net at U5.14 (D5): now also U43.2 (VOUT)
- net at U5.15 (D4): now also U42.2 (VOUT)
- net at U5.2 (D2): now also U32.2 (VOUT)
- net at U5.3 (D1): now also U23.2 (VOUT)
- net at U5.4 (D0): now also U14.2 (VOUT)
- net at U1.1 (D3): now also U33.2 (VOUT)
- net at U1.12 (D7): now also U34.2 (VOUT)
- net at U1.13 (D6): now also U25.2 (VOUT)
- net at U1.14 (D5): now also U16.2 (VOUT)
- net at U1.2 (D2): now also U24.2 (VOUT)
- net at U1.3 (D1): now also U15.2 (VOUT)
Other:
- moved on the sheet: J1, U1, U3, U4, U5, U6, U7, U8

Commit message: %50 done with PCB
Parts:
- removed U17, U27, U37, U7: A3144, A3144HallEffect:1x03_P1.50mm_Vertical_A3144HallEffect, symbol Sensor_Magnetic:A1104LLHL
- removed U2, U3, U4, U5: MUX, D16, symbol 8to1_MUX:SN74HC151DR
- added C1, C10, C11, C12, C13, C14, C15, C16, C17, C18, C19, C2, C20, C21, C22, C23, C24, C25, C26, C27, C28, C29, C3, C30, C31, C32, C33, C34, C35, C36, C37, C38, C39, C4, C40, C5, C6, C7, C8, C9: 0.1uF, footprints:CAP_CL21_SAM-M, symbol Device:C
- added C41, C42: 4.7uF, Capacitor_THT:CP_Axial_L10.0mm_D4.5mm_P15.00mm_Horizontal, symbol Device:C_Polarized_Small_US
- added IC1: LM2937ET-3.3_NOPB, ECE445L:TO254P470X1028X1955-3P, symbol ECE445L:LM2937ET-3.3_NOPB
- added R1, R10, R11, R12, R13, R14, R15, R16, R17, R18, R19, R2, R20, R21, R22, R23, R24, R25, R26, R27, R28, R29, R3, R30, R31, R32, R33, R34, R35, R36, R37, R38, R39, R4, R40, R5, R6, R7, R8, R9: 10k, ECE445L:R_Axial_DIN0204_L3.6mm_D1.6mm_P7.62mm_Horizontal, symbol Device:R
- added TP1, TP2, TP3, TP4, TP5, TP6, TP7: TP, ECE445L:Testpoint_1x02_P2.54mm, symbol ECE445L:Testpoint
- added U17, U27, U37, U7: MUX, 8to1_MUX:D16, symbol 8to1_MUX:SN74HC151DR
- added U2, U3, U4, U5: A3144, A3144HallEffect:1x03_P1.50mm_Vertical_A3144HallEffect, symbol Sensor_Magnetic:A1104LLHL
- U1: footprint D16 -> 8to1_MUX:D16
Connections:
- net 3.3V_Board: now also C42.1, IC1.3 (OUTPUT), R1.2, R10.2, R11.2, R12.2, R13.2, R14.2, R15.2, R16.2, R17.2, R18.2, R19.2, R2.2, R20.2, R21.2, R22.2, R23.2, R24.2, R25.2, R26.2, R27.2, R28.2, R29.2, R3.2, R30.2, R31.2, R32.2, R33.2, R34.2, R35.2, R36.2, R37.2, R38.2, R39.2, R4.2, R40.2, R5.2, R6.2, R7.2, R8.2, R9.2, TP7.1 (A), TP7.2 (B), U17.16 (VCC), U2.1 (VCC), U27.16 (VCC), U3.1 (VCC), U37.16 (VCC), U4.1 (VCC), U5.1 (VCC), U7.16 (VCC); no longer J1.1 (3.3V)
- net GND: now also J1.14 (GND), J1.20 (GND), J1.34 (GND), J1.39 (GND), J1.6 (GND), J1.9 (GND), C1.2, C10.2, C11.2, C12.2, C13.2, C14.2, C15.2, C16.2, C17.2, C18.2, C19.2, C2.2, C20.2, C21.2, C22.2, C23.2, C24.2, C25.2, C26.2, C27.2, C28.2, C29.2, C3.2, C30.2, C31.2, C32.2, C33.2, C34.2, C35.2, C36.2, C37.2, C38.2, C39.2, C4.2, C40.2, C41.2, C42.2, C5.2, C6.2, C7.2, C8.2, C9.2, IC1.2 (GND), TP1.2 (B), TP2.2 (B), TP3.2 (B), TP4.2 (B), TP5.2 (B), TP6.2 (B), U17.7 (*G), U17.8 (GND), U2.3 (GND), U27.7 (*G), U27.8 (GND), U3.3 (GND), U37.7 (*G), U37.8 (GND), U4.3 (GND), U5.3 (GND), U7.7 (*G), U7.8 (GND)
- net GPIO14/PIN8: now also U17.11 (A), U27.11 (A), U37.11 (A), U7.11 (A)
- net GPIO15/PIN10: now also U17.10 (B), U27.10 (B), U37.10 (B), U7.10 (B)
- net GPIO18/PIN12: now also U17.9 (C), U27.9 (C), U37.9 (C), U7.9 (C)
- net at U30.2 (VOUT): now also C27.1, R27.1, U27.2 (D2)
- net at U18.2 (VOUT): now also C17.1, R17.1, U17.4 (D0)
- net at U39.2 (VOUT): now also C34.1, R34.1, U37.3 (D1)
- net at U40.2 (VOUT): now also C35.1, R35.1, U37.2 (D2)
- net at U31.2 (VOUT): now also C28.1, R28.1, U27.1 (D3)
- net at U22.2 (VOUT): now also C21.1, R21.1, U17.15 (D4)
- net at U13.2 (VOUT): now also C14.1, R14.1, U7.14 (D5)
- net at U21.2 (VOUT): now also C20.1, R20.1, U17.1 (D3)
- net at U12.2 (VOUT): now also C13.1, R13.1, U7.15 (D4)
- net at U26.2 (VOUT): now also C24.1, R24.1, U17.12 (D7)
- net at U32.2 (VOUT): now also C29.1, R29.1, U27.15 (D4)
- net at U35.2 (VOUT): now also C31.1, R31.1, U27.13 (D6)
- net at U36.2 (VOUT): now also C32.1, R32.1, U27.12 (D7)
- net at U9.2 (VOUT): now also C10.1, R10.1, U7.3 (D1)
- net at U8.2 (VOUT): now also C9.1, R9.1, U7.4 (D0)
- net at U1.15 (D4): now also C2.1, R2.1, U2.2 (VOUT)
- net at U42.2 (VOUT): now also C37.1, R37.1, U37.15 (D4)
- net at U44.2 (VOUT): now also C39.1, R39.1, U37.13 (D6)
- net at U16.2 (VOUT): now also C16.1, R16.1, U7.12 (D7); no longer U1.14 (D5)
- net at U1.12 (D7): now also C8.1, R8.1, U5.2 (VOUT); no longer U34.2 (VOUT)
- net at U14.2 (VOUT): now also C15.1, R15.1, U7.13 (D6)
- net at U1.2 (D2), U24.2 (VOUT): now also C4.1, R4.1
- net at U11.2 (VOUT): now also C12.1, R12.1, U7.1 (D3)
- net at U29.2 (VOUT): now also C26.1, R26.1, U27.3 (D1)
- net GPIO17/PIN11: now reaches J1.11 (GPIO17)
- net GPIO17/PIN11: now also TP4.1 (A), U27.6 (W)
- net GPIO27/PIN15: now reaches J1.13 (GPIO27)
- net GPIO27/PIN15: now also TP5.1 (A), U37.6 (W)
- net 5V Board: now reaches J1.2 (5V)
- net 5V Board: now also C41.1, IC1.1 (INPUT)
- net GPIO2/PIN3: now reaches J1.3 (GPIO2)
- net GPIO2/PIN3: now also U1.6 (W), TP1.1 (A)
- net GPIO3/PIN5: now reaches J1.5 (GPIO3)
- net GPIO3/PIN5: now also TP2.1 (A), U7.6 (W)
- net GPIO4/PIN7: now reaches J1.7 (GPIO4)
- net GPIO4/PIN7: now also TP3.1 (A), U17.6 (W)
- net at U1.4 (D0), U6.2 (VOUT): now also C1.1, R1.1, TP6.1 (A)
- net at U20.2 (VOUT): now also C19.1, R19.1, U17.2 (D2)
- net at U38.2 (VOUT): now also C33.1, R33.1, U37.4 (D0)
- net at U28.2 (VOUT): now also C25.1, R25.1, U27.4 (D0)
- net at U19.2 (VOUT): now also C18.1, R18.1, U17.3 (D1)
- net at U10.2 (VOUT): now also C11.1, R11.1, U7.2 (D2)
- net at U1.1 (D3), U33.2 (VOUT): now also C5.1, R5.1
- net at U1.3 (D1), U15.2 (VOUT): now also C3.1, R3.1
- net at U23.2 (VOUT): now also C22.1, R22.1, U17.14 (D5)
- net at U41.2 (VOUT): now also C36.1, R36.1, U37.1 (D3)
- net at U45.2 (VOUT): now also C40.1, R40.1, U37.12 (D7)
- net at U43.2 (VOUT): now also C38.1, R38.1, U37.14 (D5)
- net at U1.13 (D6): now also C7.1, R7.1, U4.2 (VOUT); no longer U25.2 (VOUT)
- new net: C6.1, R6.1, U1.14 (D5), U3.2 (VOUT)
- new net: C23.1, R23.1, U17.13 (D6), U25.2 (VOUT)
- new net: C30.1, R30.1, U27.14 (D5), U34.2 (VOUT)
Other:
- moved on the sheet: J1, U6

Commit message: duck
Connections:
- net GND: now also J1.25 (GND); no longer C1.2, C10.2, C11.2, C12.2, C13.2, C14.2, C15.2, C16.2, C17.2, C18.2, C19.2, C2.2, C20.2, C21.2, C22.2, C23.2, C24.2, C25.2, C26.2, C27.2, C28.2, C29.2, C3.2, C30.2, C31.2, C32.2, C33.2, C34.2, C35.2, C36.2, C37.2, C38.2, C39.2, C4.2, C40.2, C41.2, C42.2, C5.2, C6.2, C7.2, C8.2, C9.2, IC1.2 (GND), J1.14 (GND), J1.20 (GND), J1.34 (GND), J1.39 (GND), J1.6 (GND), J1.9 (GND), TP6.2 (B), U10.3 (GND), U11.3 (GND), U12.3 (GND), U13.3 (GND), U14.3 (GND), U15.3 (GND), U16.3 (GND), U18.3 (GND), U19.3 (GND), U2.3 (GND), U20.3 (GND), U21.3 (GND), U22.3 (GND), U23.3 (GND), U24.3 (GND), U25.3 (GND), U26.3 (GND), U28.3 (GND), U29.3 (GND), U3.3 (GND), U30.3 (GND), U31.3 (GND), U32.3 (GND), U33.3 (GND), U34.3 (GND), U35.3 (GND), U36.3 (GND), U38.3 (GND), U39.3 (GND), U4.3 (GND), U40.3 (GND), U41.3 (GND), U42.3 (GND), U43.3 (GND), U44.3 (GND), U45.3 (GND), U5.3 (GND), U6.3 (GND), U8.3 (GND), U9.3 (GND)
- new net GND2: C1.2, C10.2, C11.2, C12.2, C13.2, C14.2, C15.2, C16.2, C17.2, C18.2, C19.2, C2.2, C20.2, C21.2, C22.2, C23.2, C24.2, C25.2, C26.2, C27.2, C28.2, C29.2, C3.2, C30.2, C31.2, C32.2, C33.2, C34.2, C35.2, C36.2, C37.2, C38.2, C39.2, C4.2, C40.2, C5.2, C6.2, C7.2, C8.2, C9.2, J1.39 (GND), TP6.2 (B), U10.3 (GND), U11.3 (GND), U12.3 (GND), U13.3 (GND), U14.3 (GND), U15.3 (GND), U16.3 (GND), U18.3 (GND), U19.3 (GND), U2.3 (GND), U20.3 (GND), U21.3 (GND), U22.3 (GND), U23.3 (GND), U24.3 (GND), U25.3 (GND), U26.3 (GND), U28.3 (GND), U29.3 (GND), U3.3 (GND), U30.3 (GND), U31.3 (GND), U32.3 (GND), U33.3 (GND), U34.3 (GND), U35.3 (GND), U36.3 (GND), U38.3 (GND), U39.3 (GND), U4.3 (GND), U40.3 (GND), U41.3 (GND), U42.3 (GND), U43.3 (GND), U44.3 (GND), U45.3 (GND), U5.3 (GND), U6.3 (GND), U8.3 (GND), U9.3 (GND)
- new net GND3: C41.2, C42.2, IC1.2 (GND), J1.6 (GND)
- no-connect marks 0 -> 33
